Commit message: Update robot and make it running (skidsteering robot + 2D Lidar)

File: src/skid_steer_robot/urdf/skid_robot.urdf.xacro (robot description, xacro)
@@ -1,12 +1,136 @@
 <?xml version="1.0"?>
 <robot name="skid_robot" xmlns:xacro="http://www.ros.org/wiki/xacro">
-<xacro:include filename="$(find skid_steer_robot)/urdf/lidar_2d.xacro"/>
-<xacro:include filename="$(find skid_steer_robot)/urdf/_d435.urdf.xacro"/>
-<!-- <xacro:include filename="$(find skid_steer_robot)/urdf/mono_camera.xacro"/> -->
-<xacro:include filename="$(find skid_steer_robot)/urdf/imu.xacro"/>
-<xacro:include filename="$(find skid_steer_robot)/urdf/ultrasonic.xacro"/>
-<!-- <xacro:include filename="$(find skid_steer_robot)/urdf/3d_lidar.xacro"/> -->
-<!-- Add Dummy Link  -->
-<link name="base_footprint">
+<link name="base_link">
+    <inertial>
+        <origin xyz="0.0 0.0 0.0" rpy="0.0 0.0 0.0"/>
+        <mass value="5.0"/>
+        <inertia ixx="0.0" ixy="0.0" ixz="0.0" iyy="0.0" iyz="0.0" izz="0.0"/>
+    </inertial>
+    <visual>
+        <geometry>
+            <box size="0.4 0.3 0.09"/>
+        </geometry>
+        <origin xyz="0 0 0.05"/>
+        <material name="base_link_material">
+            <color rgba="0.0 0.0 1.0 1.0"/>
+        </material>
+    </visual>
+    <collision>
+        <geometry>
+            <box size="0.4 0.3 0.09"/>
+        </geometry>
+        <origin xyz="0 0 0.05"/>
+    </collision>
+</link>
+<link name="front_right_wheel">
+  <visual>
+      <geometry>
+          <cylinder radius="0.06" length="0.02"/>
+      </geometry>
+      <origin rpy="1.5708 0 0"/>
+      <material name="">
+        <color rgba="0.0 0.0 0.0 1.0"/>
+      </material>
+  </visual>
+  <collision>
+      <geometry>
+          <cylinder radius="0.06" length="0.02"/>
+      </geometry>
+      <origin rpy="1.5708 0 0"/>
+  </collision>
+  <inertial>
+      <mass value="1.0"/>
+      <origin rpy="0 0 0"/>
+      <inertia ixx="0.001" ixy="0.0" ixz="0.0" iyy="0.001" iyz="0.0" izz="0.001"/>
+  </inertial>
+</link>
+<joint name="front_right_wheel_joint" type="continuous">
+  <parent link="base_link"/>
+  <child link="front_right_wheel"/>
+  <origin xyz="0.16 -0.16 0.05" rpy="0 0 0"/>
+  <axis xyz="0 1 0"/>
+</joint>
+<link name="front_left_wheel">
+    <visual>
+        <geometry>
+            <cylinder radius="0.06" length="0.02"/>
+        </geometry>
+        <origin rpy="1.5708 0 0"/>
+        <material name="">
+          <color rgba="0.0 0.0 0.0 1.0"/>
+        </material>
+    </visual>
+    <collision>
+        <geometry>
+            <cylinder radius="0.06" length="0.02"/>
+        </geometry>
+        <origin rpy="1.5708 0 0"/>
+    </collision>
+    <inertial>
+        <mass value="1.0"/>
+        <inertia ixx="0.001" ixy="0.0" ixz="0.0" iyy="0.001" iyz="0.0" izz="0.001"/>
+      </inertial>
+  </link>
+  <joint name="front_left_wheel_joint" type="continuous">
+    <parent link="base_link"/>
+    <child link="front_left_wheel"/>
+    <origin xyz="0.16 0.16 0.05" rpy="0 0 0"/>
+    <axis xyz="0 1 0"/>
+  </joint>
+  <link name="rear_right_wheel">
+    <visual>
+        <geometry>
+            <cylinder radius="0.06" length="0.02"/>
+        </geometry>
+        <origin rpy="1.5708 0 0"/>
+        <material name="">
+          <color rgba="0.0 0.0 0.0 1.0"/>
+        </material>
+    </visual>
+    <collision>
+        <geometry>
+            <cylinder radius="0.06" length="0.02"/>
+        </geometry>
+        <origin rpy="1.5708 0 0"/>
+    </collision>
+    <inertial>
+        <mass value="1.0"/>
+        <inertia ixx="0.001" ixy="0.0" ixz="0.0" iyy="0.001" iyz="0.0" izz="0.001"/>
+      </inertial>
+  </link>
+  <joint name="rear_right_wheel_joint" type="continuous">
+    <parent link="base_link"/>
+    <child link="rear_right_wheel"/>
+    <origin xyz="-0.16 -0.16 0.05" rpy="0 0 0"/>
+    <axis xyz="0 1 0"/>
+  </joint>
+  <link name="rear_left_wheel">
+    <visual>
+        <geometry>
+            <cylinder radius="0.06" length="0.02"/>
+        </geometry>
+        <origin rpy="1.5708 0 0"/>
+        <material name="">
+          <color rgba="0.0 0.0 0.0 1.0"/>
+        </material>
+    </visual>
+    <collision>
+        <geometry>
+            <cylinder radius="0.06" length="0.02"/>
+        </geometry>
+        <origin rpy="1.5708 0 0"/>
+    </collision>
+    <inertial>
+        <mass value="1.0"/>
+        <inertia ixx="0.001" ixy="0.0" ixz="0.0" iyy="0.001" iyz="0.0" izz="0.001"/>
+      </inertial>
+  </link>
+  <joint name="rear_left_wheel_joint" type="continuous">
+    <parent link="base_link"/>
+    <child link="rear_left_wheel"/>
+    <origin xyz="-0.16 0.16 0.05" rpy="0 0 0"/>
+    <axis xyz="0 1 0"/>
+  </joint>
+  <link name="base_footprint">
 </link>
 <joint name="base_footprint_joint" type="fixed">
@@ -17,161 +141,53 @@
     <child link ="base_link"/>
 </joint>
-   <!-- Base Link -->
-   <link name="base_link">
-    <inertial>
-        <origin xyz="0.0 0.0 0.0" rpy="0.0 0.0 0.0"/>
-        <mass value="5.0"/>
-        <inertia ixx="0.0" ixy="0.0" ixz="0.0" iyy="0.0" iyz="0.0" izz="0.0"/>
+<link name="lidar_base_link">
+    <inertial>
+      <origin xyz="0.0 0.0 0.0" rpy="0.0 0.0 0.0"/>
+      <mass value="0.5"/> <!-- Adjust mass as needed -->
+      <inertia ixx="0.0" ixy="0.0" ixz="0.0" iyy="0.0" iyz="0.0" izz="0.0"/>
     </inertial>
     <visual>
-        <geometry>
-            <box size="0.4 0.3 0.09"/>
-        </geometry>
-        <origin xyz="0 0 0.05"/>
-        <material name="base_link_material">
-            <color rgba="0.0 0.0 1.0 1.0"/>
-        </material>
-    </visual>
-    <collision>
-        <geometry>
-            <box size="0.4 0.3 0.09"/>
-        </geometry>
-        <origin xyz="0 0 0.05"/>
-    </collision>
-</link>
-    <!-- Front Right Wheel Link -->
-<link name="front_right_wheel">
-  <visual>
-      <geometry>
-          <cylinder radius="0.06" length="0.02"/>
-      </geometry>
-      <origin rpy="1.5708 0 0"/>
+      <geometry>
+        <box size="0.1 0.2 0.07"/>
+      </geometry>
+      <origin xyz="0 0 0.0"/>
       <material name="">
-        <color rgba="0.0 0.0 0.0 1.0"/>
+        <color rgba="0.0 0.0 1.0 1.0"/>
       </material>
-  </visual>
-  <collision>
-      <geometry>
-          <cylinder radius="0.06" length="0.02"/>
-      </geometry>
-      <origin rpy="1.5708 0 0"/>
-  </collision>
-  <inertial>
-      <mass value="1.0"/>
-      <origin rpy="0 0 0"/>
-      <inertia ixx="0.001" ixy="0.0" ixz="0.0" iyy="0.001" iyz="0.0" izz="0.001"/>
-  </inertial>
-</link>
-<!-- Front Right Wheel Joint -->
-<joint name="front_right_wheel_joint" type="continuous">
-  <parent link="base_link"/>
-  <child link="front_right_wheel"/>
-  <origin xyz="0.16 -0.16 0.05" rpy="0 0 0"/>
-  <axis xyz="0 1 0"/>
-</joint>
-  <!-- Front Left Wheel Link -->
-  <link name="front_left_wheel">
-    <visual>
-        <geometry>
-            <cylinder radius="0.06" length="0.02"/>
-        </geometry>
-        <origin rpy="1.5708 0 0"/>
-        <material name="">
-          <color rgba="0.0 0.0 0.0 1.0"/>
-        </material>
-    </visual>
-    <collision>
-        <geometry>
-            <cylinder radius="0.06" length="0.02"/>
-        </geometry>
-        <origin rpy="1.5708 0 0"/>
-    </collision>
-    <inertial>
-        <mass value="1.0"/>
-        <inertia ixx="0.001" ixy="0.0" ixz="0.0" iyy="0.001" iyz="0.0" izz="0.001"/>
-      </inertial>
-  </link>
-  <!-- Front Left Wheel Joint -->
-  <joint name="front_left_wheel_joint" type="continuous">
-    <parent link="base_link"/>
-    <child link="front_left_wheel"/>
-    <origin xyz="0.16 0.16 0.05" rpy="0 0 0"/>
-    <axis xyz="0 1 0"/>
-  </joint>
-   <!-- Rear Right Wheel Link -->
-   <link name="rear_right_wheel">
-    <visual>
-        <geometry>
-            <cylinder radius="0.06" length="0.02"/>
-        </geometry>
-        <origin rpy="1.5708 0 0"/>
-        <material name="">
-          <color rgba="0.0 0.0 0.0 1.0"/>
-        </material>
-    </visual>
-    <collision>
-        <geometry>
-            <cylinder radius="0.06" length="0.02"/>
-        </geometry>
-        <origin rpy="1.5708 0 0"/>
-    </collision>
-    <inertial>
-        <mass value="1.0"/>
-        <inertia ixx="0.001" ixy="0.0" ixz="0.0" iyy="0.001" iyz="0.0" izz="0.001"/>
-      </inertial>
-  </link>
-  <!-- rear Right Wheel Joint -->
-  <joint name="rear_right_wheel_joint" type="continuous">
-    <parent link="base_link"/>
-    <child link="rear_right_wheel"/>
-    <origin xyz="-0.16 -0.16 0.05" rpy="0 0 0"/>
-    <axis xyz="0 1 0"/>
-  </joint>
-   <!-- Rear Left Wheel Link -->
-   <link name="rear_left_wheel">
-    <visual>
-        <geometry>
-            <cylinder radius="0.06" length="0.02"/>
-        </geometry>
-        <origin rpy="1.5708 0 0"/>
-        <material name="">
-          <color rgba="0.0 0.0 0.0 1.0"/>
-        </material>
-    </visual>
-    <collision>
-        <geometry>
-            <cylinder radius="0.06" length="0.02"/>
-        </geometry>
-        <origin rpy="1.5708 0 0"/>
-    </collision>
-    <inertial>
-        <mass value="1.0"/>
-        <inertia ixx="0.001" ixy="0.0" ixz="0.0" iyy="0.001" iyz="0.0" izz="0.001"/>
-      </inertial>
-  </link>
-  <!-- rear Left Wheel Joint -->
-  <joint name="rear_left_wheel_joint" type="continuous">
-    <parent link="base_link"/>
-    <child link="rear_left_wheel"/>
-    <origin xyz="-0.16 0.16 0.05" rpy="0 0 0"/>
-    <axis xyz="0 1 0"/>
-  </joint>
-<xacro:sensor_d435 parent="base_link" use_nominal_extrinsics="true">
-  <origin xyz="0.19 0 0.1" rpy="0 0 0"/>
-</xacro:sensor_d435>
-<!-- Skid-Steer Drive Plugin -->
+    </visual>
+    <collision>
+      <geometry>
+        <box size="0.2 0.2 0.07"/>
+      </geometry>
+      <origin xyz="0 0 0.3"/> <!-- Adjust position as needed -->
+    </collision>
+  </link>
+  <joint name="lidar_base_joint" type="fixed">
+    <parent link="base_link"/>
+    <child link="lidar_base_link"/>
+    <origin xyz="-0.1 0 0.1" rpy="0 0 0"/> <!-- Adjust height as needed -->
+  </joint>
 <gazebo>
   <plugin name="skid_steer_drive_controller" filename="libgazebo_ros_skid_steer_drive.so">
+    <!-- Update rate of the plugin in Hz -->
     <updateRate>100.0</updateRate>
+    <!-- Namespace for the robot in ROS -->
     <robotNamespace>/</robotNamespace>
+    <!-- Names of the joints controlling each wheel -->
     <leftFrontJoint>front_left_wheel_joint</leftFrontJoint>
     <rightFrontJoint>front_right_wheel_joint</rightFrontJoint>
     <leftRearJoint>rear_left_wheel_joint</leftRearJoint>
     <rightRearJoint>rear_right_wheel_joint</rightRearJoint>
+    <!-- Distance between the front and rear wheels -->
     <wheelSeparation>0.34</wheelSeparation>
+    <!-- Diameter of the wheels -->
     <wheelDiameter>0.12</wheelDiameter>
+    <!-- Frame of reference for the robot's base -->
     <robotBaseFrame>base_footprint</robotBaseFrame>
+    <!-- Maximum torque applied to the wheels -->
     <torque>20</torque>
+    <!-- ROS topic for receiving velocity commands -->
     <topicName>cmd_vel</topicName>
+    <!-- Whether to broadcast the transform from the base frame to the wheels -->
     <broadcastTF>false</broadcastTF>
     <commandTopic>cmd_vel</commandTopic>
@@ -183,18 +199,54 @@
   </plugin>
 </gazebo>
-<gazebo reference="front_left_wheel">
-  <material>Gazebo/Black</material>
-</gazebo>
-<gazebo reference="front_right_wheel">
-  <material>Gazebo/Black</material>
-</gazebo>
-<gazebo reference="rear_left_wheel">
-  <material>Gazebo/Black</material>
-</gazebo>
-<gazebo reference="rear_right_wheel">
-  <material>Gazebo/Black</material>
-</gazebo>
-<gazebo reference="base_link">
-  <material>Gazebo/Blue</material>
+<!-- LIDAR Sensor -->
+    <gazebo reference="lidar_base_link">
+    <!-- Define a sensor of type "ray" (commonly used for LiDAR sensors) -->
+    <sensor type="ray" name="lidar_sensor">
+        <!-- Set the pose of the sensor relative to the link it's attached to (x, y, z, roll, pitch, yaw) -->
+        <pose>0 0 0 0 0 0</pose>
+        <!-- Enable or disable visualization of the sensor in Gazebo -->
+        <visualize>true</visualize>
+        <!-- Set the update rate for the sensor in Hz (how often it produces data) -->
+        <update_rate>40</update_rate>
+        <!-- Define the ray properties of the sensor (LiDAR emits rays to measure distances) -->
+        <ray>
+            <scan>
+                <horizontal>
+                    <!-- Number of samples (rays) per scan -->
+                    <samples>720</samples>
+                    <!-- Resolution of the scan (typically 1 means 1 ray per angle unit) -->
+                    <resolution>1</resolution>
+                    <!-- Minimum angle of the scan (in radians, -π/2 for a 180-degree scan) -->
+                    <min_angle>-1.570796</min_angle>
+                    <!-- Maximum angle of the scan (in radians, π/2 for a 180-degree scan) -->
+                    <max_angle>1.570796</max_angle>
+                </horizontal>
+            </scan>
+            <range>
+                <!-- Minimum range (distance) the sensor can detect -->
+                <min>0.10</min>
+                <!-- Maximum range (distance) the sensor can detect -->
+                <max>30.0</max>
+                <!-- Resolution of the distance measurements (smallest measurable distance change) -->
+                <resolution>0.01</resolution>
+            </range>
+            <!-- Define noise characteristics for the sensor -->
+            <noise>
+                <!-- Type of noise (Gaussian noise is commonly used for sensors) -->
+                <type>gaussian</type>
+                <!-- Mean value of the noise (0.0 means no bias) -->
+                <mean>0.0</mean>
+                <!-- Standard deviation of the noise (how much variation there is) -->
+                <stddev>0.01</stddev>
+            </noise>
+        </ray>
+        <!-- Attach a Gazebo plugin to simulate the LiDAR sensor in ROS -->
+        <plugin name="gazebo_ros_laser" filename="libgazebo_ros_laser.so">
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