Commit message: Add lidar Sensor and reading

File: src/skid_steer_robot/urdf/skid_robot.urdf.xacro (robot description, xacro)
@@ -1,74 +1,76 @@
 <?xml version="1.0"?>
-<robot name="skid_robot" xmlns:xacro="http://www.ros.org/wiki/xacro">
-<link name="base_link">
-    <inertial>
-        <origin xyz="0.0 0.0 0.0" rpy="0.0 0.0 0.0"/>
-        <mass value="5.0"/>
-        <inertia ixx="0.0" ixy="0.0" ixz="0.0" iyy="0.0" iyz="0.0" izz="0.0"/>
-    </inertial>
-    <visual>
-        <geometry>
-            <box size="0.4 0.3 0.09"/>
-        </geometry>
-        <origin xyz="0 0 0.05"/>
-        <material name="base_link_material">
-            <color rgba="0.0 0.0 1.0 1.0"/>
-        </material>
-    </visual>
-    <collision>
-        <geometry>
-            <box size="0.4 0.3 0.09"/>
-        </geometry>
-        <origin xyz="0 0 0.05"/>
-    </collision>
-</link>
-<link name="front_right_wheel">
-  <visual>
-      <geometry>
-          <cylinder radius="0.06" length="0.02"/>
-      </geometry>
-      <origin rpy="1.5708 0 0"/>
-      <material name="">
-        <color rgba="0.0 0.0 0.0 1.0"/>
-      </material>
-  </visual>
-  <collision>
-      <geometry>
-          <cylinder radius="0.06" length="0.02"/>
-      </geometry>
-      <origin rpy="1.5708 0 0"/>
-  </collision>
-  <inertial>
+<robot name="skid_robot"
+  xmlns:xacro="http://www.ros.org/wiki/xacro">
+  <!-- Robot essentials -->
+  <link name="base_link">
+    <inertial>
+      <origin xyz="0.0 0.0 0.0" rpy="0.0 0.0 0.0"/>
+      <mass value="5.0"/>
+      <inertia ixx="0.0" ixy="0.0" ixz="0.0" iyy="0.0" iyz="0.0" izz="0.0"/>
+    </inertial>
+    <visual>
+      <geometry>
+        <box size="0.4 0.3 0.09"/>
+      </geometry>
+      <origin xyz="0 0 0.05"/>
+      <material name="base_link_material">
+        <color rgba="0.0 0.0 1.0 1.0"/>
+      </material>
+    </visual>
+    <collision>
+      <geometry>
+        <box size="0.4 0.3 0.09"/>
+      </geometry>
+      <origin xyz="0 0 0.05"/>
+    </collision>
+  </link>
+  <link name="front_right_wheel">
+    <visual>
+      <geometry>
+        <cylinder radius="0.06" length="0.02"/>
+      </geometry>
+      <origin rpy="1.5708 0 0"/>
+      <material name="">
+        <color rgba="0.0 0.0 0.0 1.0"/>
+      </material>
+    </visual>
+    <collision>
+      <geometry>
+        <cylinder radius="0.06" length="0.02"/>
+      </geometry>
+      <origin rpy="1.5708 0 0"/>
+    </collision>
+    <inertial>
       <mass value="1.0"/>
       <origin rpy="0 0 0"/>
       <inertia ixx="0.001" ixy="0.0" ixz="0.0" iyy="0.001" iyz="0.0" izz="0.001"/>
-  </inertial>
-</link>
-<joint name="front_right_wheel_joint" type="continuous">
-  <parent link="base_link"/>
-  <child link="front_right_wheel"/>
-  <origin xyz="0.16 -0.16 0.05" rpy="0 0 0"/>
-  <axis xyz="0 1 0"/>
-</joint>
-<link name="front_left_wheel">
-    <visual>
-        <geometry>
-            <cylinder radius="0.06" length="0.02"/>
-        </geometry>
-        <origin rpy="1.5708 0 0"/>
-        <material name="">
-          <color rgba="0.0 0.0 0.0 1.0"/>
-        </material>
-    </visual>
-    <collision>
-        <geometry>
-            <cylinder radius="0.06" length="0.02"/>
-        </geometry>
-        <origin rpy="1.5708 0 0"/>
-    </collision>
-    <inertial>
-        <mass value="1.0"/>
-        <inertia ixx="0.001" ixy="0.0" ixz="0.0" iyy="0.001" iyz="0.0" izz="0.001"/>
-      </inertial>
+    </inertial>
+  </link>
+  <joint name="front_right_wheel_joint" type="continuous">
+    <parent link="base_link"/>
+    <child link="front_right_wheel"/>
+    <origin xyz="0.16 -0.16 0.05" rpy="0 0 0"/>
+    <axis xyz="0 1 0"/>
+  </joint>
+  <link name="front_left_wheel">
+    <visual>
+      <geometry>
+        <cylinder radius="0.06" length="0.02"/>
+      </geometry>
+      <origin rpy="1.5708 0 0"/>
+      <material name="">
+        <color rgba="0.0 0.0 0.0 1.0"/>
+      </material>
+    </visual>
+    <collision>
+      <geometry>
+        <cylinder radius="0.06" length="0.02"/>
+      </geometry>
+      <origin rpy="1.5708 0 0"/>
+    </collision>
+    <inertial>
+      <mass value="1.0"/>
+      <inertia ixx="0.001" ixy="0.0" ixz="0.0" iyy="0.001" iyz="0.0" izz="0.001"/>
+    </inertial>
   </link>
   <joint name="front_left_wheel_joint" type="continuous">
@@ -80,22 +82,22 @@
   <link name="rear_right_wheel">
     <visual>
-        <geometry>
-            <cylinder radius="0.06" length="0.02"/>
-        </geometry>
-        <origin rpy="1.5708 0 0"/>
-        <material name="">
-          <color rgba="0.0 0.0 0.0 1.0"/>
-        </material>
-    </visual>
-    <collision>
-        <geometry>
-            <cylinder radius="0.06" length="0.02"/>
-        </geometry>
-        <origin rpy="1.5708 0 0"/>
-    </collision>
-    <inertial>
-        <mass value="1.0"/>
-        <inertia ixx="0.001" ixy="0.0" ixz="0.0" iyy="0.001" iyz="0.0" izz="0.001"/>
-      </inertial>
+      <geometry>
+        <cylinder radius="0.06" length="0.02"/>
+      </geometry>
+      <origin rpy="1.5708 0 0"/>
+      <material name="">
+        <color rgba="0.0 0.0 0.0 1.0"/>
+      </material>
+    </visual>
+    <collision>
+      <geometry>
+        <cylinder radius="0.06" length="0.02"/>
+      </geometry>
+      <origin rpy="1.5708 0 0"/>
+    </collision>
+    <inertial>
+      <mass value="1.0"/>
+      <inertia ixx="0.001" ixy="0.0" ixz="0.0" iyy="0.001" iyz="0.0" izz="0.001"/>
+    </inertial>
   </link>
   <joint name="rear_right_wheel_joint" type="continuous">
@@ -107,22 +109,22 @@
   <link name="rear_left_wheel">
     <visual>
-        <geometry>
-            <cylinder radius="0.06" length="0.02"/>
-        </geometry>
-        <origin rpy="1.5708 0 0"/>
-        <material name="">
-          <color rgba="0.0 0.0 0.0 1.0"/>
-        </material>
-    </visual>
-    <collision>
-        <geometry>
-            <cylinder radius="0.06" length="0.02"/>
-        </geometry>
-        <origin rpy="1.5708 0 0"/>
-    </collision>
-    <inertial>
-        <mass value="1.0"/>
-        <inertia ixx="0.001" ixy="0.0" ixz="0.0" iyy="0.001" iyz="0.0" izz="0.001"/>
-      </inertial>
+      <geometry>
+        <cylinder radius="0.06" length="0.02"/>
+      </geometry>
+      <origin rpy="1.5708 0 0"/>
+      <material name="">
+        <color rgba="0.0 0.0 0.0 1.0"/>
+      </material>
+    </visual>
+    <collision>
+      <geometry>
+        <cylinder radius="0.06" length="0.02"/>
+      </geometry>
+      <origin rpy="1.5708 0 0"/>
+    </collision>
+    <inertial>
+      <mass value="1.0"/>
+      <inertia ixx="0.001" ixy="0.0" ixz="0.0" iyy="0.001" iyz="0.0" izz="0.001"/>
+    </inertial>
   </link>
   <joint name="rear_left_wheel_joint" type="continuous">
@@ -133,16 +135,17 @@
   </joint>
   <link name="base_footprint">
-</link>
-<joint name="base_footprint_joint" type="fixed">
-      <origin
-        xyz="0.0 0.0 0.0"
-        rpy="0 0 0" />
+  </link>
+  <joint name="base_footprint_joint" type="fixed">
+    <origin xyz="0.0 0.0 0.0" rpy="0 0 0" />
     <parent link ="base_footprint"/>
     <child link ="base_link"/>
-</joint>
-<link name="lidar_base_link">
-    <inertial>
-      <origin xyz="0.0 0.0 0.0" rpy="0.0 0.0 0.0"/>
-      <mass value="0.5"/> <!-- Adjust mass as needed -->
+  </joint>
+  <!-- Robot essentials -->
+  <!-- Base lidar link -->
+  <link name="lidar_base_link">
+    <inertial>
+      <origin xyz="0.0 0.0 0.0" rpy="0.0 0.0 0.0"/>
+      <mass value="0.5"/>
+      <!-- Adjust mass as needed -->
       <inertia ixx="0.0" ixy="0.0" ixz="0.0" iyy="0.0" iyz="0.0" izz="0.0"/>
     </inertial>
@@ -160,93 +163,134 @@
         <box size="0.2 0.2 0.07"/>
       </geometry>
-      <origin xyz="0 0 0.3"/> <!-- Adjust position as needed -->
-    </collision>
-  </link>
+      <origin xyz="0 0 0.3"/>
+      <!-- Adjust position as needed -->
+    </collision>
+  </link>
+  <!-- Base Lidar Joint -->
   <joint name="lidar_base_joint" type="fixed">
     <parent link="base_link"/>
     <child link="lidar_base_link"/>
-    <origin xyz="-0.1 0 0.1" rpy="0 0 0"/> <!-- Adjust height as needed -->
-  </joint>
-<gazebo>
-  <plugin name="skid_steer_drive_controller" filename="libgazebo_ros_skid_steer_drive.so">
-    <!-- Update rate of the plugin in Hz -->
-    <updateRate>100.0</updateRate>
-    <!-- Namespace for the robot in ROS -->
-    <robotNamespace>/</robotNamespace>
-    <!-- Names of the joints controlling each wheel -->
-    <leftFrontJoint>front_left_wheel_joint</leftFrontJoint>
-    <rightFrontJoint>front_right_wheel_joint</rightFrontJoint>
-    <leftRearJoint>rear_left_wheel_joint</leftRearJoint>
-    <rightRearJoint>rear_right_wheel_joint</rightRearJoint>
-    <!-- Distance between the front and rear wheels -->
-    <wheelSeparation>0.34</wheelSeparation>
-    <!-- Diameter of the wheels -->
-    <wheelDiameter>0.12</wheelDiameter>
-    <!-- Frame of reference for the robot's base -->
-    <robotBaseFrame>base_footprint</robotBaseFrame>
-    <!-- Maximum torque applied to the wheels -->
-    <torque>20</torque>
-    <!-- ROS topic for receiving velocity commands -->
-    <topicName>cmd_vel</topicName>
-    <!-- Whether to broadcast the transform from the base frame to the wheels -->
-    <broadcastTF>false</broadcastTF>
-    <commandTopic>cmd_vel</commandTopic>
-    <odometryTopic>odom</odometryTopic>
-    <odometryFrame>odom</odometryFrame>
-    <covariance_x>0.000100</covariance_x>
-    <covariance_y>0.000100</covariance_y>
-    <covariance_yaw>0.010000</covariance_yaw>
-  </plugin>
-</gazebo>
-<!-- LIDAR Sensor -->
-    <gazebo reference="lidar_base_link">
+    <origin xyz="-0.1 0 0.1" rpy="0 0 0"/>
+    <!-- Adjust height as needed -->
+  </joint>
+  <!-- Lidar link -->
+  <link name="lidar_link">
+    <inertial>
+      <origin xyz="0.0 0.0 0.0" rpy="0.0 0.0 0.0"/>
+      <mass value="0.0"/>
+      <inertia ixx="1.0" ixy="0.0" ixz="0.0" iyy="1.0" iyz="0.0" izz="1.0"/>
+    </inertial>
+    <visual name="lidar_link_visual">
+      <origin xyz="0.0 0.0 0.0" rpy="0.0 0.0 0"/>
+      <geometry>
+        <mesh filename="package://skid_steer_robot/meshes/2d_lidar.STL"/>
+      </geometry>
+      <material name="">
+        <color rgba="0.0 0.0 0.0 1.0"/>
+        <texture filename=""/>
+      </material>
+    </visual>
+    <collision>
+      <origin xyz="0.0 0.0 0.0" rpy="0.0 0.0 0.0"/>
+      <geometry>
+        <mesh filename="package://skid_steer_robot/meshes/2d_lidar.STL"/>
+      </geometry>
+    </collision>
+  </link>
+  <!-- Lidar Joint -->
+  <joint name="lidar_joint" type="fixed">
+    <axis xyz="0 1 0" />
+    <origin xyz="0 0 0.06" rpy="0 0 0"/>
+    <parent link="lidar_base_link"/>
+    <child link="lidar_link"/>
+  </joint>
+  <!-- Motion Plugin -->
+  <gazebo>
+    <plugin name="skid_steer_drive_controller" filename="libgazebo_ros_skid_steer_drive.so">
+      <!-- Update rate of the plugin in Hz -->
+      <updateRate>100.0</updateRate>
+      <!-- Namespace for the robot in ROS -->
+      <robotNamespace>/</robotNamespace>
+      <!-- Names of the joints controlling each wheel -->
+      <leftFrontJoint>front_left_wheel_joint</leftFrontJoint>
+      <rightFrontJoint>front_right_wheel_joint</rightFrontJoint>
+      <leftRearJoint>rear_left_wheel_joint</leftRearJoint>
+      <rightRearJoint>rear_right_wheel_joint</rightRearJoint>
+      <!-- Distance between the front and rear wheels -->
+      <wheelSeparation>0.34</wheelSeparation>
+      <!-- Diameter of the wheels -->
+      <wheelDiameter>0.12</wheelDiameter>
+      <!-- Frame of reference for the robot's base -->
+      <robotBaseFrame>base_footprint</robotBaseFrame>
+      <!-- Maximum torque applied to the wheels -->
+      <torque>20</torque>
+      <!-- ROS topic for receiving velocity commands -->
+      <topicName>cmd_vel</topicName>
+      <!-- Whether to broadcast the transform from the base frame to the wheels -->
+      <broadcastTF>false</broadcastTF>
+      <commandTopic>cmd_vel</commandTopic>
+      <odometryTopic>odom</odometryTopic>
+      <odometryFrame>odom</odometryFrame>
+      <covariance_x>0.000100</covariance_x>
+      <covariance_y>0.000100</covariance_y>
+      <covariance_yaw>0.010000</covariance_yaw>
+    </plugin>
+  </gazebo>
+  <!-- LIDAR Sensor -->
+  <gazebo reference="lidar_link">
     <!-- Define a sensor of type "ray" (commonly used for LiDAR sensors) -->
     <sensor type="ray" name="lidar_sensor">
-        <!-- Set the pose of the sensor relative to the link it's attached to (x, y, z, roll, pitch, yaw) -->
-        <pose>0 0 0 0 0 0</pose>
-        <!-- Enable or disable visualization of the sensor in Gazebo -->
-        <visualize>true</visualize>
-        <!-- Set the update rate for the sensor in Hz (how often it produces data) -->
-        <update_rate>40</update_rate>
-        <!-- Define the ray properties of the sensor (LiDAR emits rays to measure distances) -->
-        <ray>
-            <scan>
-                <horizontal>
-                    <!-- Number of samples (rays) per scan -->
-                    <samples>720</samples>
-                    <!-- Resolution of the scan (typically 1 means 1 ray per angle unit) -->
-                    <resolution>1</resolution>
-                    <!-- Minimum angle of the scan (in radians, -π/2 for a 180-degree scan) -->
-                    <min_angle>-1.570796</min_angle>
-                    <!-- Maximum angle of the scan (in radians, π/2 for a 180-degree scan) -->
-                    <max_angle>1.570796</max_angle>
-                </horizontal>
-            </scan>
-            <range>
-                <!-- Minimum range (distance) the sensor can detect -->
-                <min>0.10</min>
-                <!-- Maximum range (distance) the sensor can detect -->
-                <max>30.0</max>
-                <!-- Resolution of the distance measurements (smallest measurable distance change) -->
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
Commit message: Add Camera

File: src/skid_steer_robot/urdf/skid_robot.urdf.xacro (robot description, xacro)
@@ -204,4 +204,24 @@
     <parent link="lidar_base_link"/>
     <child link="lidar_link"/>
+  </joint>
+  <!-- Camera -->
+  <link name="mono_camera_link">
+    <visual>
+      <geometry>
+        <box size="0.03 0.03 0.03"/>
+      </geometry>
+      <material name=""/>
+    </visual>
+    <collision>
+      <geometry>
+        <box size="0.03 0.03 0.03"/>
+      </geometry>
+    </collision>
+  </link>
+  <joint name="mono_camera_joint" type="fixed">
+    <origin xyz="0.2 0.0 0.06" rpy="1.57 0 0"/>
+    <parent link="base_link"/>
+    <child link="mono_camera_link"/>
+    <axis xyz="0.0 0.0 0.0"/>
   </joint>
   <!-- Motion Plugin -->
@@ -294,3 +314,68 @@
     <material>Gazebo/Black</material>
   </gazebo>
+  <!-- Camera Plugin-->
+  <gazebo reference="mono_camera_link">
+    <!-- Defines the sensor type and name. The sensor is attached to the camera_link_optical reference -->
+    <sensor type="camera" name="camera">
+      <!-- The pose of the camera relative to the reference frame. It includes position (x, y, z) and orientation (roll, pitch, yaw) -->
+      <pose>0 0 0 -1.57 0 0</pose>
+      <!-- The update rate in Hz for how often the camera captures images -->
+      <update_rate>30.0</update_rate>
+      <!-- Whether to visualize the camera sensor in the Gazebo GUI -->
+      <visualize>true</visualize>
+      <!-- Camera-specific parameters -->
+      <camera name="head">
+        <!-- The horizontal field of view (in radians) of the camera -->
+        <horizontal_fov>1.3962634</horizontal_fov>
+        <!-- Image properties -->
+        <image>
+          <!-- Width of the captured image in pixels -->
+          <width>800</width>
+          <!-- Height of the captured image in pixels -->
+          <height>800</height>
+          <!-- Format of the image. 'L8' means an 8-bit grayscale image (mono format) -->
+          <format>L8</format>
+        </image>
+        <!-- Clipping planes define the near and far boundaries for rendering objects in the camera's view -->
+        <clip>
+          <!-- Minimum distance at which objects are rendered -->
+          <near>0.02</near>
+          <!-- Maximum distance at which objects are rendered -->
+          <far>300</far>
+        </clip>
+        <!-- Noise settings for simulating realistic sensor noise -->
+        <noise>
+          <!-- Type of noise to apply, in this case, Gaussian noise -->
+          <type>gaussian</type>
+          <!-- The mean value of the noise (center of the Gaussian distribution) -->
+          <mean>0.0</mean>
+          <!-- The standard deviation of the noise (spread of the Gaussian distribution) -->
+          <stddev>0.007</stddev>
+        </noise>
+      </camera>
+      <!-- Plugin to interface the camera with ROS -->
+      <plugin name="camera_controller" filename="libgazebo_ros_camera.so">
+        <!-- Whether the camera is always on -->
+        <alwaysOn>true</alwaysOn>
+        <!-- The update rate for the plugin. '0.0' means it updates as fast as possible -->
+        <updateRate>0.0</updateRate>
+        <!-- The ROS topic name for the camera images -->
+        <cameraName>/mybot/camera</cameraName>
+        <!-- The ROS topic name for the image data (mono format) -->
+        <imageTopicName>image_mono</imageTopicName>
+        <!-- The ROS topic name for the camera info (camera parameters) -->
+        <cameraInfoTopicName>camera_info_mono</cameraInfoTopicName>
+        <!-- The name of the reference frame associated with the camera -->
+        <frameName>mono_camera_link</frameName>
+        <!-- The baseline distance for stereo cameras, irrelevant for mono but sometimes required for plugin configuration -->
+        <hackBaseline>0.07</hackBaseline>
+        <!-- Distortion parameters for camera lens distortion correction (all set to 0.0, indicating no distortion) -->
+        <distortionK1>0.0</distortionK1>
+        <distortionK2>0.0</distortionK2>
+        <distortionK3>0.0</distortionK3>
+        <distortionT1>0.0</distortionT1>
+        <distortionT2>0.0</distortionT2>
+      </plugin>
+    </sensor>
+  </gazebo>
 </robot>

Commit message: Add IMU sensor

File: src/skid_steer_robot/urdf/skid_robot.urdf.xacro (robot description, xacro)
@@ -379,3 +379,47 @@
     </sensor>
   </gazebo>
+  <joint name="imu_sensor_joint" type="fixed">
+        <axis xyz="0 0 1" />
+        <origin xyz="0.4 0.0 0.06" rpy="0 0 0"/>
+        <parent link="base_link"/>
+        <child link="imu_sensor_link"/>
+    </joint>
+    <link name="imu_sensor_link">
+        <collision>
+            <origin xyz="0 0 0" rpy="0 0 0"/>
+            <geometry>
+                <box size="0.02 0.02 0.02"/>
+            </geometry>
+        </collision>
+        <visual>
+            <origin xyz="0 0 0" rpy="0 0 0"/>
+            <geometry>
+                <box size="0.02 0.02 0.02"/>
+            </geometry>
+            <material name=""/>
+        </visual>
+        <inertial>
+            <mass value="0.001" />
+            <origin xyz="0 0 0" rpy="0 0 0"/>
+            <inertia ixx="0.00000015" ixy="0" ixz="0" iyy="0.00000015" iyz="0" izz="0.00000015" />
+        </inertial>
+    </link>
+    <gazebo reference="imu_sensor_link">
+        <gravity>true</gravity>
+        <sensor name='imu_sensor' type='imu'>
+            <always_on>1</always_on>
+            <update_rate>1000</update_rate>
+            <visualize>1</visualize>
+            <topic>__default_topic__</topic>
+            <plugin name='imu_plugin' filename='libgazebo_ros_imu_sensor.so'>
+                <topicName>imu_data</topicName>
+                <bodyName>imu_sensor_link</bodyName>
+                <updateRateHZ>10.0</updateRateHZ>
+                <gaussianNoise>0.0</gaussianNoise>
+                <xyzOffset>0 0 0</xyzOffset>
+                <rpyOffset>0 0 0</rpyOffset>
+            </plugin>
+            <pose>0 0 0 0 0 0</pose>
+        </sensor>
+    </gazebo>
 </robot>

Commit message: Fix and add IMU (position + frame)

File: src/skid_steer_robot/urdf/skid_robot.urdf.xacro (robot description, xacro)
@@ -105,4 +105,5 @@
     <child link="rear_right_wheel"/>
     <origin xyz="-0.16 -0.16 0.05" rpy="0 0 0"/>
+    <limit effort="100" velocity="100"/>
     <axis xyz="0 1 0"/>
   </joint>
@@ -397,5 +398,7 @@
                 <box size="0.02 0.02 0.02"/>
             </geometry>
-            <material name=""/>
+                        <material name="red_material">
+                <color rgba="1.0 0.0 0.0 1.0"/> <!-- Red color, fully opaque -->
+            </material>
         </visual>
         <inertial>
@@ -409,8 +412,9 @@
         <sensor name='imu_sensor' type='imu'>
             <always_on>1</always_on>
-            <update_rate>1000</update_rate>
-            <visualize>1</visualize>
+            <update_rate>30</update_rate>
+            <visualize>true</visualize>
             <topic>__default_topic__</topic>
             <plugin name='imu_plugin' filename='libgazebo_ros_imu_sensor.so'>
+                <frameName>imu_sensor_link</frameName>
                 <topicName>imu_data</topicName>
                 <bodyName>imu_sensor_link</bodyName>

Commit message: Change lidar to 360deg + fix imu position

File: src/skid_steer_robot/urdf/skid_robot.urdf.xacro (robot description, xacro)
@@ -273,11 +273,11 @@
           <horizontal>
             <!-- Number of samples (rays) per scan -->
-            <samples>720</samples>
+            <samples>360</samples>
             <!-- Resolution of the scan (typically 1 means 1 ray per angle unit) -->
             <resolution>1</resolution>
             <!-- Minimum angle of the scan (in radians, -π/2 for a 180-degree scan) -->
-            <min_angle>-1.570796</min_angle>
+            <min_angle>-3.14159</min_angle>
             <!-- Maximum angle of the scan (in radians, π/2 for a 180-degree scan) -->
-            <max_angle>1.570796</max_angle>
+            <max_angle>3.14159</max_angle>
           </horizontal>
         </scan>
@@ -382,5 +382,5 @@
   <joint name="imu_sensor_joint" type="fixed">
         <axis xyz="0 0 1" />
-        <origin xyz="0.4 0.0 0.06" rpy="0 0 0"/>
+        <origin xyz="0.0 0.0 0.1" rpy="0 0 0"/>
         <parent link="base_link"/>
         <child link="imu_sensor_link"/>
@@ -399,5 +399,5 @@
             </geometry>
                         <material name="red_material">
-                <color rgba="1.0 0.0 0.0 1.0"/> <!-- Red color, fully opaque -->
+                <color rgba="1.0 0.0 0.0 1.0"/>
             </material>
         </visual>

Commit message: Center lidar for accurate obstacle range

File: src/skid_steer_robot/urdf/skid_robot.urdf.xacro (robot description, xacro)
@@ -172,5 +172,5 @@
     <parent link="base_link"/>
     <child link="lidar_base_link"/>
-    <origin xyz="-0.1 0 0.1" rpy="0 0 0"/>
+    <origin xyz="-0.0 0 0.1" rpy="0 0 0"/>
     <!-- Adjust height as needed -->
   </joint>
@@ -382,5 +382,5 @@
   <joint name="imu_sensor_joint" type="fixed">
         <axis xyz="0 0 1" />
-        <origin xyz="0.0 0.0 0.1" rpy="0 0 0"/>
+        <origin xyz="0.18 0.0 0.1" rpy="0 0 0"/>
         <parent link="base_link"/>
         <child link="imu_sensor_link"/>
