Commit message: Add transmissions and tune parameters for robot wheels

File: src/skid_steer_robot/urdf/skid_robot.urdf.xacro (robot description, xacro)
@@ -53,4 +53,15 @@
     <axis xyz="0 1 0"/>
   </joint>
+  <!-- Transmissions -->
+  <transmission name="front_right_wheel_trans">
+    <type>transmission_interface/SimpleTransmission</type>
+    <joint name="front_right_wheel_joint">
+      <hardwareInterface>hardware_interface/VelocityJointInterface</hardwareInterface>
+    </joint>
+    <actuator name="front_right_wheel_motor">
+    <hardwareInterface>hardware_interface/VelocityJointInterface</hardwareInterface>
+      <mechanicalReduction>1</mechanicalReduction>
+    </actuator>
+  </transmission>
   <link name="front_left_wheel">
     <visual>
@@ -80,4 +91,15 @@
     <axis xyz="0 1 0"/>
   </joint>
+  <!-- Transmissions -->
+  <transmission name="front_left_wheel_trans">
+    <type>transmission_interface/SimpleTransmission</type>
+    <joint name="front_left_wheel_joint">
+      <hardwareInterface>hardware_interface/VelocityJointInterface</hardwareInterface>
+    </joint>
+    <actuator name="front_left_wheel_motor">
+    <hardwareInterface>hardware_interface/VelocityJointInterface</hardwareInterface>
+      <mechanicalReduction>1</mechanicalReduction>
+    </actuator>
+  </transmission>
   <link name="rear_right_wheel">
     <visual>
@@ -108,4 +130,15 @@
     <axis xyz="0 1 0"/>
   </joint>
+  <!-- Transmissions -->
+  <transmission name="rear_right_wheel_trans">
+    <type>transmission_interface/SimpleTransmission</type>
+    <joint name="rear_right_wheel_joint">
+      <hardwareInterface>hardware_interface/VelocityJointInterface</hardwareInterface>
+    </joint>
+    <actuator name="rear_right_wheel_motor">
+    <hardwareInterface>hardware_interface/VelocityJointInterface</hardwareInterface>
+      <mechanicalReduction>1</mechanicalReduction>
+    </actuator>
+  </transmission>
   <link name="rear_left_wheel">
     <visual>
@@ -135,4 +168,15 @@
     <axis xyz="0 1 0"/>
   </joint>
+  <!-- Transmissions -->
+  <transmission name="rear_left_wheel_trans">
+    <type>transmission_interface/SimpleTransmission</type>
+    <joint name="rear_left_wheel_joint">
+        <hardwareInterface>hardware_interface/VelocityJointInterface</hardwareInterface>
+    </joint>
+    <actuator name="rear_left_wheel_motor">
+      <hardwareInterface>hardware_interface/VelocityJointInterface</hardwareInterface>
+      <mechanicalReduction>1</mechanicalReduction>
+    </actuator>
+  </transmission>
   <link name="base_footprint">
   </link>
@@ -142,4 +186,25 @@
     <child link ="base_link"/>
   </joint>
+  <!-- new  -->
+    <gazebo reference="rear_right_wheel">
+      <mu1 value="1.5"/>
+      <mu2 value="1.5"/>
+      <material>Gazebo/Red</material>
+    </gazebo>
+    <gazebo reference="rear_left_wheel">
+      <mu1 value="1.5"/>
+      <mu2 value="1.5"/>
+      <material>Gazebo/Red</material>
+    </gazebo>
+    <gazebo reference="front_right_wheel">
+      <mu1 value="1.5"/>
+      <mu2 value="1.5"/>
+      <material>Gazebo/Red</material>
+    </gazebo>
+    <gazebo reference="front_left_wheel">
+      <mu1 value="1.5"/>
+      <mu2 value="1.5"/>
+      <material>Gazebo/Red</material>
+    </gazebo>
   <!-- Robot essentials -->
   <!-- Base lidar link -->

Commit message: Still trying to fix the wheels frames

File: src/skid_steer_robot/urdf/skid_robot.urdf.xacro (robot description, xacro)
@@ -2,4 +2,15 @@
 <robot name="skid_robot"
   xmlns:xacro="http://www.ros.org/wiki/xacro">
+  <xacro:property name="wheel_kp" value="1000000.0" />
+  <xacro:property name="wheel_kd" value="100.0" />
+  <xacro:property name="wheel_mu1" value="100" />
+  <xacro:property name="wheel_mu2" value="100" />
+  <xacro:property name="wheel_slip1" value="0.5" />
+  <xacro:property name="wheel_slip2" value="0" />
+    <xacro:macro name="cylinder_inertia" params="m r h">
+    <inertia ixx="${m*(3*r*r+h*h)/12}" ixy="0" ixz="0"
+             iyy="${m*(3*r*r+h*h)/12}" iyz="0"
+             izz="${m*r*r/2}" />
+  </xacro:macro>
   <!-- Robot essentials -->
   <link name="base_link">
@@ -40,9 +51,23 @@
       </geometry>
       <origin rpy="1.5708 0 0"/>
+      <surface>
+        <friction>
+          <fdir1>1 0 0</fdir1>
+          <kp>${wheel_kp}</kp> <!-- kp and kd for rubber -->
+          <kd>${wheel_kd}</kd>
+          <mu>${wheel_mu1}</mu>
+          <mu2>${wheel_mu2}</mu2>
+          <slip1>${wheel_slip1}</slip1>
+          <slip2>${wheel_slip2}</slip2>
+        </friction>
+      </surface>
     </collision>
     <inertial>
       <mass value="1.0"/>
-      <origin rpy="0 0 0"/>
-      <inertia ixx="0.001" ixy="0.0" ixz="0.0" iyy="0.001" iyz="0.0" izz="0.001"/>
+      <!-- <origin rpy="0 0 0"/>
+      <inertia ixx="0.001" ixy="0.0" ixz="0.0" iyy="0.001" iyz="0.0" izz="0.001"/> -->
+      <inertia ixx="0.00833" ixy="0" ixz="0"
+              iyy="0.00833" iyz="0"
+              izz="0.005" />
     </inertial>
   </link>
@@ -52,4 +77,5 @@
     <origin xyz="0.16 -0.16 0.05" rpy="0 0 0"/>
     <axis xyz="0 1 0"/>
+    <limit lower="0" upper="6.28" effort="100" velocity="10"/>
   </joint>
   <!-- Transmissions -->
@@ -57,8 +83,8 @@
     <type>transmission_interface/SimpleTransmission</type>
     <joint name="front_right_wheel_joint">
-      <hardwareInterface>hardware_interface/VelocityJointInterface</hardwareInterface>
+      <hardwareInterface>hardware_interface/EffortJointInterface</hardwareInterface>
     </joint>
     <actuator name="front_right_wheel_motor">
-    <hardwareInterface>hardware_interface/VelocityJointInterface</hardwareInterface>
+      <hardwareInterface>hardware_interface/EffortJointInterface</hardwareInterface>
       <mechanicalReduction>1</mechanicalReduction>
     </actuator>
@@ -79,8 +105,22 @@
       </geometry>
       <origin rpy="1.5708 0 0"/>
+      <surface>
+        <friction>
+          <fdir1>1 0 0</fdir1>
+          <kp>${wheel_kp}</kp> <!-- kp and kd for rubber -->
+          <kd>${wheel_kd}</kd>
+          <mu>${wheel_mu1}</mu>
+          <mu2>${wheel_mu2}</mu2>
+          <slip1>${wheel_slip1}</slip1>
+          <slip2>${wheel_slip2}</slip2>
+        </friction>
+      </surface>
     </collision>
     <inertial>
       <mass value="1.0"/>
-      <inertia ixx="0.001" ixy="0.0" ixz="0.0" iyy="0.001" iyz="0.0" izz="0.001"/>
+      <!-- <inertia ixx="0.001" ixy="0.0" ixz="0.0" iyy="0.001" iyz="0.0" izz="0.001"/> -->
+        <inertia ixx="0.00833" ixy="0" ixz="0"
+           iyy="0.00833" iyz="0"
+           izz="0.005" />
     </inertial>
   </link>
@@ -90,4 +130,5 @@
     <origin xyz="0.16 0.16 0.05" rpy="0 0 0"/>
     <axis xyz="0 1 0"/>
+    <limit lower="0" upper="6.28" effort="100" velocity="10"/>
   </joint>
   <!-- Transmissions -->
@@ -117,8 +158,22 @@
       </geometry>
       <origin rpy="1.5708 0 0"/>
+      <surface>
+        <friction>
+          <fdir1>1 0 0</fdir1>
+          <kp>${wheel_kp}</kp> <!-- kp and kd for rubber -->
+          <kd>${wheel_kd}</kd>
+          <mu>${wheel_mu1}</mu>
+          <mu2>${wheel_mu2}</mu2>
+          <slip1>${wheel_slip1}</slip1>
+          <slip2>${wheel_slip2}</slip2>
+        </friction>
+      </surface>
     </collision>
     <inertial>
       <mass value="1.0"/>
-      <inertia ixx="0.001" ixy="0.0" ixz="0.0" iyy="0.001" iyz="0.0" izz="0.001"/>
+      <!-- <inertia ixx="0.001" ixy="0.0" ixz="0.0" iyy="0.001" iyz="0.0" izz="0.001"/> -->
+        <inertia ixx="0.00833" ixy="0" ixz="0"
+           iyy="0.00833" iyz="0"
+           izz="0.005" />
     </inertial>
   </link>
@@ -129,4 +184,5 @@
     <limit effort="100" velocity="100"/>
     <axis xyz="0 1 0"/>
+    <limit lower="0" upper="6.28" effort="100" velocity="10"/>
   </joint>
   <!-- Transmissions -->
@@ -156,8 +212,22 @@
       </geometry>
       <origin rpy="1.5708 0 0"/>
+      <surface>
+        <friction>
+          <fdir1>1 0 0</fdir1>
+          <kp>${wheel_kp}</kp> <!-- kp and kd for rubber -->
+          <kd>${wheel_kd}</kd>
+          <mu>${wheel_mu1}</mu>
+          <mu2>${wheel_mu2}</mu2>
+          <slip1>${wheel_slip1}</slip1>
+          <slip2>${wheel_slip2}</slip2>
+        </friction>
+      </surface>
     </collision>
     <inertial>
       <mass value="1.0"/>
-      <inertia ixx="0.001" ixy="0.0" ixz="0.0" iyy="0.001" iyz="0.0" izz="0.001"/>
+      <!-- <inertia ixx="0.001" ixy="0.0" ixz="0.0" iyy="0.001" iyz="0.0" izz="0.001"/> -->
+        <inertia ixx="0.00833" ixy="0" ixz="0"
+           iyy="0.00833" iyz="0"
+           izz="0.005" />
     </inertial>
   </link>
@@ -167,4 +237,5 @@
     <origin xyz="-0.16 0.16 0.05" rpy="0 0 0"/>
     <axis xyz="0 1 0"/>
+    <limit lower="0" upper="6.28" effort="100" velocity="10"/>
   </joint>
   <!-- Transmissions -->
@@ -468,5 +539,5 @@
         </visual>
         <inertial>
-            <mass value="0.001" />
+            <mass value="0.1" />
             <origin xyz="0 0 0" rpy="0 0 0"/>
             <inertia ixx="0.00000015" ixy="0" ixz="0" iyy="0.00000015" iyz="0" izz="0.00000015" />

Commit message: Improvment trying to find a solution for the wheels rotation!

File: src/skid_steer_robot/urdf/skid_robot.urdf.xacro (robot description, xacro)
@@ -128,5 +128,5 @@
     <parent link="base_link"/>
     <child link="front_left_wheel"/>
-    <origin xyz="0.16 0.16 0.05" rpy="0 0 0"/>
+    <origin xyz="0.16 0.16 0.02" rpy="0 0 0"/>
     <axis xyz="0 1 0"/>
     <limit lower="0" upper="6.28" effort="100" velocity="10"/>
@@ -181,5 +181,5 @@
     <parent link="base_link"/>
     <child link="rear_right_wheel"/>
-    <origin xyz="-0.16 -0.16 0.05" rpy="0 0 0"/>
+    <origin xyz="-0.16 -0.16 0.02" rpy="0 0 0"/>
     <limit effort="100" velocity="100"/>
     <axis xyz="0 1 0"/>
@@ -235,5 +235,5 @@
     <parent link="base_link"/>
     <child link="rear_left_wheel"/>
-    <origin xyz="-0.16 0.16 0.05" rpy="0 0 0"/>
+    <origin xyz="-0.16 0.16 0.02" rpy="0 0 0"/>
     <axis xyz="0 1 0"/>
     <limit lower="0" upper="6.28" effort="100" velocity="10"/>
@@ -253,5 +253,5 @@
   </link>
   <joint name="base_footprint_joint" type="fixed">
-    <origin xyz="0.0 0.0 0.0" rpy="0 0 0" />
+    <origin xyz="0.0 0.0 0.02" rpy="0 0 0" />
     <parent link ="base_footprint"/>
     <child link ="base_link"/>
@@ -366,5 +366,5 @@
     <plugin name="skid_steer_drive_controller" filename="libgazebo_ros_skid_steer_drive.so">
       <!-- Update rate of the plugin in Hz -->
-      <updateRate>30.0</updateRate>
+      <updateRate>100.0</updateRate>
       <!-- Namespace for the robot in ROS -->
       <robotNamespace>/</robotNamespace>
@@ -381,5 +381,5 @@
       <robotBaseFrame>base_footprint</robotBaseFrame>
       <!-- Maximum torque applied to the wheels -->
-      <torque>20</torque>
+      <torque>50</torque>
       <!-- ROS topic for receiving velocity commands -->
       <topicName>cmd_vel</topicName>

Commit message: Urdf improvmet (still working on wheels  tf rotation)

File: src/skid_steer_robot/urdf/skid_robot.urdf.xacro (robot description, xacro)
@@ -4,6 +4,6 @@
   <xacro:property name="wheel_kp" value="1000000.0" />
   <xacro:property name="wheel_kd" value="100.0" />
-  <xacro:property name="wheel_mu1" value="100" />
-  <xacro:property name="wheel_mu2" value="100" />
+  <xacro:property name="wheel_mu1" value="1000" />
+  <xacro:property name="wheel_mu2" value="1000" />
   <xacro:property name="wheel_slip1" value="0.5" />
   <xacro:property name="wheel_slip2" value="0" />
@@ -61,4 +61,9 @@
           <slip2>${wheel_slip2}</slip2>
         </friction>
+        <contact>
+          <ode>
+            <min_depth>0.003</min_depth>
+          </ode>
+        </contact>
       </surface>
     </collision>
@@ -77,5 +82,4 @@
     <origin xyz="0.16 -0.16 0.05" rpy="0 0 0"/>
     <axis xyz="0 1 0"/>
-    <limit lower="0" upper="6.28" effort="100" velocity="10"/>
   </joint>
   <!-- Transmissions -->
@@ -115,4 +119,9 @@
           <slip2>${wheel_slip2}</slip2>
         </friction>
+        <contact>
+          <ode>
+            <min_depth>0.003</min_depth>
+          </ode>
+        </contact>
       </surface>
     </collision>
@@ -130,5 +139,4 @@
     <origin xyz="0.16 0.16 0.02" rpy="0 0 0"/>
     <axis xyz="0 1 0"/>
-    <limit lower="0" upper="6.28" effort="100" velocity="10"/>
   </joint>
   <!-- Transmissions -->
@@ -168,4 +176,9 @@
           <slip2>${wheel_slip2}</slip2>
         </friction>
+        <contact>
+          <ode>
+            <min_depth>0.003</min_depth>
+          </ode>
+        </contact>
       </surface>
     </collision>
@@ -184,5 +197,4 @@
     <limit effort="100" velocity="100"/>
     <axis xyz="0 1 0"/>
-    <limit lower="0" upper="6.28" effort="100" velocity="10"/>
   </joint>
   <!-- Transmissions -->
@@ -222,4 +234,9 @@
           <slip2>${wheel_slip2}</slip2>
         </friction>
+        <contact>
+          <ode>
+            <min_depth>0.003</min_depth>
+          </ode>
+        </contact>
       </surface>
     </collision>
@@ -237,5 +254,4 @@
     <origin xyz="-0.16 0.16 0.02" rpy="0 0 0"/>
     <axis xyz="0 1 0"/>
-    <limit lower="0" upper="6.28" effort="100" velocity="10"/>
   </joint>
   <!-- Transmissions -->
